File: MR2/_autosave-MR1.sch (KiCad schematic (older format))
At the start: 16 parts, among them J1 Conn_01x04_Male, J2 Conn_01x04_Male, J3 Conn_01x04_Male, J4 Conn_01x04_Male, J5 Conn_01x02_Male, J6 Conn_01x04_Male, J7 Conn_01x04_Male, J8 Conn_01x04_Male, Q1 2SC1815, U5 LPC1768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

Commit message: update:MR1の基板完成
Connections:
- no-connect marks 19 -> 18
Changed lines of the file:
@@
 Text Label 1550 4450 0    50   ~ 0
 tape_led
-NoConn ~ 2450 5550
 $EndSCHEMATC
